Commit message: map in orde gemaakt w seppe de goat

File: webots_ros2_brick/install/webots_ros2_brick/share/webots_ros2_brick/resource/brick.urdf (robot description, URDF)
Before this commit: robot BRICKV1, 0 links, 0 joints
Links:
- added link base_link; collision box size=0.5 0.3 0.1; visual box size=0.5 0.3 0.1
